Commit message: edit

File: install/ur_simulation_gz/share/ur_simulation_gz/urdf/ur_gz.urdf.xacro (robot description, xacro)
@@ -59,5 +59,5 @@
     force_abs_paths="true"
     >
-    <origin xyz="0 0 0" rpy="0 0 0" />          <!-- position robot in the world -->
+    <origin xyz="0 0 0.1" rpy="0 0 0" />          <!-- position robot in the world -->
   </xacro:ur_robot>
   <gazebo reference="world">
